Commit message: modifed and running

File: pterotactyl/objects/test_objects/0.obj.urdf (robot description, URDF)
Before this commit: robot object.urdf, 1 links, 0 joints
Links:
- link baseLink: geometry collision mesh filename=/home/robospare/suddhu/active-touch/pterotactyl/objects/tes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 scale=1 1 1; visual mesh filename=/home/robospare/suddhu/active-touch/pterotactyl/objects/tes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 scale=1 1 1
